Commit message: test

File: src/ros1_wiki/forklift/urdf/forklift.urdf.xacro (robot description, xacro)
@@ -6,5 +6,13 @@
             <origin xyz="0.0 0.0 0.0" rpy="0.0 0.0 0.0"/>
             <mass value="50.0"/>
-            <inertia ixx="0.0" ixy="0.0" ixz="0.0" iyy="0.0" iyz="0.0" izz="0.0"/>
+            <!--
+            <inertia ixx="0.05" ixy="0.05" ixz="0.05" iyy="1.3419385416666667" iyz="1.3419385416666667" izz="2.296875"/>
+            -->
+            <inertia ixx="1.3419385416666667"
+                iyy="1.3419385416666667"
+                izz="2.296875"
+                ixy="0.0"
+                ixz="0.0"
+                iyz="0.0"/>
         </inertial>
         <visual name="">
@@ -23,6 +31,19 @@
                 <box size="0.525 0.525 0.2155"/>
             </geometry>
+            <!--
+            <surface>
+                <friction>
+                    <ode>
+                        <mu>100</mu>
+                        <mu2>100</mu2>
+                    </ode>
+                </friction>
+            </surface>
+            -->
         </collision>
     </link>
+    <gazebo reference="base_link">
+        <material>Gazebo/Blue</material>
+    </gazebo>
     <joint name="base_joint" type="fixed">
         <origin xyz="0.0 0.0 0.0" rpy="0.0 0.0 0.0"/>
@@ -36,5 +57,15 @@
                 <origin xyz="0.0 0.0 0.0" rpy="0.0 0.0 0.0"/>
                 <mass value="1.0"/>
-                <inertia ixx="0.0" ixy="0.0" ixz="0.0" iyy="0.0" iyz="0.0" izz="0.0"/>        </inertial>
+                <!--
+                <inertia ixx="0.05" ixy="0.05" ixz="0.05"
+                    iyy="0.0009333333333333333" iyz="0.0009333333333333333" izz="0.0018"/>
+                -->
+                <inertia ixx="0.0009333333333333333"
+                    iyy="0.0009333333333333333"
+                    izz="0.0018"
+                    ixy="0.0"
+                    ixz="0.0"
+                    iyz="0.0"/>
+                </inertial>
             <visual name="">
                 <origin xyz="0.0 0.0 0.0" rpy="0.0 0.0 0.0"/>
@@ -52,6 +83,19 @@
                     <cylinder radius="0.06" length="0.02"/>
                 </geometry>
+                <!--
+                <surface>
+                    <friction>
+                        <ode>
+                            <mu>100</mu>
+                            <mu2>100</mu2>
+                        </ode>
+                    </friction>
+                </surface>
+                -->
             </collision>
         </link>
+        <gazebo reference="wheel_link_${name}">
+            <material>Gazebo/Black</material>
+        </gazebo>
         <joint name="wheel_joint_${name}" type="continuous">
             <origin xyz="${x} ${y} -0.100250" rpy="1.57 0.0 0.0"/>
@@ -67,5 +111,14 @@
                 <origin xyz="0.0 0.0 0.0" rpy="0.0 0.0 0.0"/>
                 <mass value="0.5"/>
-                <inertia ixx="0.0" ixy="0.0" ixz="0.0" iyy="0.0" iyz="0.0" izz="0.0"/>
+                <!--
+                <inertia ixx="0.05" ixy="0.05" ixz="0.05"
+                    iyy="0.0005208333333333334" iyz="0.0004208333333333334" izz="0.00010833333333333334"/>
+                    -->
+                <inertia ixx="0.0005208333333333334"
+                    iyy="0.0004208333333333334"
+                    izz="0.00010833333333333334"
+                    ixy="0.0"
+                    ixz="0.0"
+                    iyz="0.0"/>
             </inertial>
             <visual name="">
@@ -86,4 +139,7 @@
             </collision>
         </link>
+        <gazebo reference="forkbase_link_${name}">
+            <material>Gazebo/Green</material>
+        </gazebo>
         <joint name="forkbase_link_${name}" type="fixed">
             <origin xyz="0.2675 ${y} -0.10025" rpy="0.0 0.0 0.0"/>
@@ -98,5 +154,14 @@
                 <origin xyz="0.0 0.0 0.0" rpy="0.0 0.0 0.0"/>
                 <mass value="0.5"/>
-                <inertia ixx="0.0" ixy="0.0" ixz="0.0" iyy="0.0" iyz="0.0" izz="0.0"/>
+                <!--
+                <inertia ixx="0.05" ixy="0.05" ixz="0.05"
+                    iyy="0.00010833333333333334" iyz="0.0026083333333333336" izz="0.0027083333333333334"/>
+                -->
+                <inertia ixx="0.00010833333333333334"
+                    iyy="0.0026083333333333336"
+                    izz="0.0027083333333333334"
+                    ixy="0.0"
+                    ixz="0.0"
+                    iyz="0.0"/>
             </inertial>
             <visual name="">
@@ -117,4 +182,7 @@
             </collision>
         </link>
+        <gazebo reference="fork_link_${name}">
+            <material>Gazebo/Green</material>
+        </gazebo>
         <joint name="fork_link_${name}" type="fixed">
             <origin xyz="0.13 0 -0.045" rpy="0.0 0.0 0.0"/>
@@ -123,6 +191,13 @@
         </joint>
     </xacro:macro>
+    <xacro:include filename="$(find realsense2_description)/urdf/_d435.urdf.xacro" />
 <!--   ***   combine component   ***   -->
-    <xacro:wheel name="back_right" x="-0.272513" y ="-0.272513"/>
+<!--
+    <xacro:wheel name="back_right" x="-0.150000" y ="-0.272513"/>
+    <xacro:wheel name="back_left" x="-0.150000" y ="0.272513"/>
+    <xacro:wheel name="front_right" x="0.150000" y ="-0.272513"/>
+    <xacro:wheel name="front_left" x="0.150000" y ="0.272513"/>
+-->
+    <xacro:wheel name="back_right" x="-0.150000" y ="-0.272513"/>
     <xacro:wheel name="back_left" x="-0.150000" y ="0.272513"/>
     <xacro:wheel name="front_right" x="0.150000" y ="-0.272513"/>

File: src/ros1_wiki/pallet/urdf/pallet.urdf.xacro (robot description, xacro)
@@ -7,6 +7,11 @@
             <inertial>
                 <origin xyz="0.0 0.0 0.0" rpy="0.0 0.0 0.0"/>
-                <mass value="0.0"/>
-                <inertia ixx="0.0" ixy="0.0" ixz="0.0" iyy="0.0" iyz="0.0" izz="0.0"/>
+                <mass value="0.1"/>
+                <inertia ixx="0.0005209083333333333"
+                    iyy="0.0007752833333333334"
+                    izz="0.0012960416666666667"
+                    ixy="0.0"
+                    ixz="0.0"
+                    iyz="0.0"/>
             </inertial>
             <visual name="">
@@ -38,6 +43,11 @@
             <inertial>
                 <origin xyz="0.0 0.0 0.0" rpy="0.0 0.0 0.0"/>
-                <mass value="0.0"/>
-                <inertia ixx="0.0" ixy="0.0" ixz="0.0" iyy="0.0" iyz="0.0" izz="0.0"/>
+                <mass value="0.01"/>
+                <inertia ixx="0.00000194"
+                    iyy="0.00000404"
+                    izz="0.00000331"
+                    ixy="0.0"
+                    ixz="0.0"
+                    iyz="0.0"/>
             </inertial>
             <visual name="">

Commit message: test

File: src/ros1_wiki/forklift/urdf/forklift.urdf.xacro (robot description, xacro)
@@ -192,4 +192,7 @@
     </xacro:macro>
     <xacro:include filename="$(find realsense2_description)/urdf/_d435.urdf.xacro" />
+    <xacro:sensor_d435 name="camera" topics_ns="camera" parent="base_link" publish_pointcloud="true">
+        <origin xyz="0.2625 0 -0.10775" rpy="0 0 0" />
+    </xacro:sensor_d435>
 <!--   ***   combine component   ***   -->
 <!--
